File: design/Power.sch (KiCad schematic (older format))
At the start: 47 parts, among them U2 TC2117, U3 DRV8302

Commit message: Implemented some improvements in schematic, but layout is completely new.
Changes in schematic:
- 3.3V or 5V CAN transceiver can be used
- DRV8301 can also be used and configured via SPI
- JTAG connector changed
- Fixed pinning of P1
- Some additional decoupling and/or filtering of analog signals
- Improved buck design according TI Webench recommendation
- Changed some component values
- maybe others...

Changes in layout:
- completely new layout
- placement of the big components is unchanged
- CAN connector rotated by 180°
- kept one layer free as a good GND plane
- many traces should be shorter and have lower impedance now
- improved buck layout

Other changes:
- updated gerber files
- updated PDFs (schematic and component placement)
- deleted all outdated files except libraries and datasheets
Parts:
- removed C25, C33: 100u, w_smd_cap:c_tant_B, symbol CP1-RESCUE-BLDC_4
- removed C51: 15u, 100v, w_smd_cap:c_2220, symbol C-RESCUE-BLDC_4
- removed C52: 2.2u, CRF1:SMD-0603_c, symbol C-RESCUE-BLDC_4
- removed D5: TVS 5V, w_smd_diode:do214ac, symbol DIODE
- added C25, C47, C48, C50: 100n, CRF1:SMD-0603_c, symbol C-RESCUE-BLDC_4
- added C33: 2.2u, CRF1:SMD-0603_c, symbol C-RESCUE-BLDC_4
- added C45: 6n8 opt, CRF1:SMD-0603_c, symbol C-RESCUE-BLDC_4
- added C46: 47u,10V, w_smd_cap:c_1210, symbol C-RESCUE-BLDC_4
- added D5: TVS 5V, Diodes_SMD:SMA_Standard, symbol TVS
- added JP3: JUMPER3, open-project:S_JUMPER_3, symbol JUMPER3
- added L2: L, CRF1:SMD-0603_r, symbol L
- added R14: 0R, CRF1:SMD-0603_r, symbol R-RESCUE-BLDC_4
- C1, C39, C40, C43, C44, C49, C8, C9: value 10u,50V -> 10u,63V; footprint CRF1:SMD-1206 -> w_smd_cap:c_1210; Part# (none) -> GRM32ER71J106KA12
- C18: value 2.2u -> 4.7u,25V; Part# (none) -> GRM188R61E475KE15
- C19: value 120p -> 1p5
- C20, C23: value 2.2u -> 2.2u,16V; Part# (none) -> GRM188R61C225KAAD
- C21: value 6.8n -> 2n
- C24: Part# (none) -> GRM188R61C225KAAD or GRM188C81A225KAAD
- C34, C36: value 2.2n -> 2n
- C37: value 15u,100V -> 22u,63V; Part# (none) -> KRM55WR71J226MH01
- D4: value DIODESCH -> Schottky; footprint Diodes_SMD:SMA_Handsoldering -> Diodes_SMD:SMA_Standard
- L1: value 22u -> 33u; footprint w_smd_inductors:inductor_smd_8x5mm -> pikim:inductor_smd_6x6mm
- R17: value 18k -> 52k5
- R18: value 3k3 -> 10k
- R19: value 15k -> 100k
- R21: value 220k -> 301k
- R48, R49, R50, R51: value 100R -> 120R
- U3: value DRV8302 -> DRV8301/2; footprint CRF1:TSSOP-56-PP -> pikim:TSSOP-56-PP
Connections:
- net labels added: DRV_MISO, DRV_MOSI, DRV_NSS, DRV_SCK
- wire segments 186 -> 174
- no-connect marks 4 -> 3
Other:
- note added: "100n in parallel would be\ngood here, but there was\nno space on the board."
- note added: "6n8 for soft-start\nrecommended."
- note added: "Bridge 2-3 for DRV8301.\nBridge 1-2 for DRV8302."
- note added: "Buck design by TI-Webench:\n7V..60V in, 5V/1.4A out\n(2015-12-30)."
- note added: "C51; 22u,63V,2220\nwas here, but there\nwas no more space."
- note added: "Mount R14 for DRV8301.\nMount R25 for DRV8302."
- note added: "Should not be needed with\nproper buck design, but is\nkept, just in case..."
- moved on the sheet: C1, C18, C19, C20, C21, C23, C24, C34, C36, C37, C39, C40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
