File: design/temp.sch (KiCad schematic (older format))
At the start: 3 parts

Commit message: Implemented some improvements in schematic, but layout is completely new.
Changes in schematic:
- 3.3V or 5V CAN transceiver can be used
- DRV8301 can also be used and configured via SPI
- JTAG connector changed
- Fixed pinning of P1
- Some additional decoupling and/or filtering of analog signals
- Improved buck design according TI Webench recommendation
- Changed some component values
- maybe others...

Changes in layout:
- completely new layout
- placement of the big components is unchanged
- CAN connector rotated by 180°
- kept one layer free as a good GND plane
- many traces should be shorter and have lower impedance now
- improved buck layout

Other changes:
- updated gerber files
- updated PDFs (schematic and component placement)
- deleted all outdated files except libraries and datasheets
Parts:
- C41: Part# (none) -> GRM188R61C225KAAD or GRM188C81A225KAAD
Changed lines of the file:
@@
 EESchema Schematic File Version 2
-LIBS:BLDC_4-rescue
 LIBS:power
 LIBS:device
@@
 LIBS:contrib
 LIBS:valves
-LIBS:crf_1
 LIBS:BLDC_4-cache
 EELAYER 25 0
@@
 encoding utf-8
 Sheet 3 7
-Title "BLDC Driver 4.11"
-Date "21 aug 2015"
-Rev "4.11"
+Title "BLDC Driver 4.11p"
+Date "2016-01-06"
+Rev "A"
 Comp "Benjamin Vedder"
-Comment1 ""
+Comment1 "modified by pikim"
 Comment2 ""
 Comment3 ""
@@
 F 2 "CRF1:SMD-0603_c" H 4188 3950 30  0001 C CNN
 F 3 "" H 4150 4100 60  0000 C CNN
+F 4 "GRM188R61C225KAAD or GRM188C81A225KAAD" H 4150 4100 60  0001 C CNN "Part#"
 	1    4150 4100
 	1    0    0    -1
